File: hardware/pcb/chip_module.kicad_pcb (KiCad board)
At the start: 4 copper layers, 85 x 50 mm, 48 parts, among them J1 Samtec LSHM-130, Q1 AO3401A, Q10 AO3400A, Q11 AO3400A, Q12 AO3400A, Q13 AO3400A, Q14 AO3400A, Q15 AO3400A, Q16 AO3400A, Q2 AO3401A, Q3 AO3401A, Q4 AO3401A, Q5 AO3401A, Q6 AO3401A, Q7 AO3401A, Q8 AO3401A, Q9 AO3400A, U1 ADG732BCPZ, U2 ADG732BCPZ, U3 ADA4530-1, U4 74LVC1G04, U5 QSSC_Chip, U6 74HCT240, U7 74HCT240

Commit message: hardware , pending to finish routes and some connections in pcb
Routing:
- net emitter_rows0: track 79.6 -> 0.00 mm, vias 2 -> 0
- net emitter_rows2: track 76.8 -> 0.00 mm, vias 2 -> 0
- net emitter_cathode7: track 58.2 -> 0.00 mm
- net emitter_anode2: track 56.6 -> 0.00 mm, vias 2 -> 0
- net emitter_cathode0: track 46.5 -> 0.00 mm
- net TIA_IN: track 34.5 -> 0.00 mm
- net col_sink6: track 32.7 -> 0.00 mm, vias 2 -> 0
- net col_sink4: track 32.3 -> 0.00 mm, vias 2 -> 0
- net col_sink7: track 30.7 -> 0.00 mm
- net col_sink1: track 27.1 -> 0.00 mm, vias 2 -> 0
- net MUX_EN2: track 26.3 -> 0.00 mm, vias 2 -> 0
- net +5V: track 24.4 -> 0.00 mm
- net row_gate1: track 23.7 -> 0.00 mm, vias 2 -> 0
- net DET_IN39: track 18.8 -> 0.00 mm
- net GND: vias 32 -> 0
- removed copper zone on In2.Cu, net +3V3
- removed copper zone on B.Cu, net GND
- removed copper zone on F.Cu, net GND
- removed copper zone on In1.Cu, net GND
Other:
- copper layers 4 -> 6
