File: hardware/pcb/qssc.kicad_sch (KiCad schematic)
At the start: 581 parts, among them J1 FT232RL, J10 USB-C, J2 5V Barrel, J3 SMA, J7 RESET, J8 MW_GATE, J9 JTAG, Q0 AO3401A, Q1 AO3401A, Q10 AO3401A, Q11 AO3401A, Q12 AO3401A, Q13 AO3401A, Q14 AO3401A, Q15 AO3401A, Q16 AO3401A, Q17 AO3401A, Q18 AO3401A, Q19 AO3401A, Q2 AO3401A, Q20 AO3401A, Q21 AO3401A, Q22 AO3401A, Q23 AO3401A, Q24 AO3401A, Q25 AO3401A, Q26 AO3401A, Q27 AO3401A, Q28 AO3401A, Q29 AO3401A, Q3 AO3401A, Q30 AO3401A, Q31 AO3401A, Q32 AO3401A, Q33 AO3401A, Q34 AO3401A, Q35 AO3401A, Q36 AO3401A, Q37 AO3401A, Q38 AO3401A, Q39 AO3401A, Q4 AO3401A, Q40 AO3401A, Q41 AO3401A, Q42 AO3401A, Q43 AO3401A, Q44 AO3401A, Q45 AO3401A, Q46 AO3401A, Q47 AO3401A, Q48 AO3401A, Q49 AO3401A, Q5 AO3401A, Q50 AO3401A, Q51 AO3401A, Q52 AO3401A, Q53 AO3401A, Q54 AO3401A, Q55 AO3401A, Q56 AO3401A, Q57 AO3401A, Q58 AO3401A, Q59 AO3401A, Q6 AO3401A, Q60 AO3401A, Q61 AO3401A, Q62 AO3401A, Q63 AO3401A, Q7 AO3401A, Q8 AO3401A, Q9 AO3401A, U1 XC7A35T-1CSG324C, U3 ADF4351BCPZ, U5 GVA-84+, U8 W25Q128JVSIQ, Y1 100MHz TCXO

Commit message: pcb: raise emitter anode to +12V_EMIT, fix DRC 43->2 (TLC5947 headroom)
Task #22: the CQD EL turn-on is 4-8 V per the fabrication protocol, so the
old +5V anode rail left the TLC5947 constant-current sink no headroom. Add a
separate +12V_EMIT LED supply (J4 barrel + F2 1A PTC + C85/C86 decoupling)
-- TLC5947 OUT pins tolerate 33 V, textbook separate-supply application.

- gen_qssc_kicad: EM_ANODE die pad +5V -> +12V_EMIT; move the EM_ANODE pad
  off the bottom edge (where its 1.0 mm width + fanout via collided with
  emitter_cat dog-bone vias 30-33) to the LEFT edge at (-10,0), clear of
  both DET/EM dog-bone fields. Reposition C85/C86 next to the new anode
  fanout. Add +12V_EMIT/+12V_EMIT_IN nets, power syms, PWR_FLAGs.
- route_signals: _is_chip_net bug fix (emitter_anode -> emitter_cat) so the
  64 cathode fanout nets now get the 0.10 mm Chip netclass; add the two
  +12V nets to POWER_NETS / POWER_ROUTER_LAYER (B.Cu).
- route_qssc_pcb: add +12V nets to STRAGGLER_POWER_NETS; fix hole_near_hole
  -- the GND stitching-via grid skipped same-net pads, so it co-located
  drills (actual 0.0 mm) on UE1's HTSSOP thermal-pad PTH vias. Add a PTH
  flag to the pads obstacle tuple and require clearance from same-net PTH
  pads so stitching vias sit OFF the pad instead of on its hole.
- tlc5947_ctrl.v: comment -- anode rail is +12V_EMIT (was +5V).
- gen_bom.py: BOM regenerator (394 comps -> 48 line items, no two-board
  leftovers); regenerate BOM.csv with the +12V_EMIT parts.

DRC on the routed merged board: 43 violations -> 2 (both Chip-clearance
between adjacent dog-bone escapes on In3.Cu -- the dense HDI case the line
router struggles with, slated for the FreeRouting pass, Task #17). The
+12V_EMIT/emitter_cat shorts, the +5V/+3V3/GND shorting_items, and all six
hole_near_hole violations are resolved.

Co-Authored-By: Claude Code <noreply@anthropic.com>
Parts:
- removed Cub0, Cub1, Cub2, Cub3, Cub4, Cub5, Cub6, Cub7: 100nF, Capacitor_SMD:C_0603_1608Metric, symbol qssc:C
- removed Q0, Q1, Q10, Q11, Q12, Q13, Q14, Q15, Q16, Q17, Q18, Q19, Q2, Q20, Q21, Q22, Q23, Q24, Q25, Q26, Q27, Q28, Q29, Q3, Q30, Q31, Q32, Q33, Q34, Q35, Q36, Q37, Q38, Q39, Q4, Q40, Q41, Q42, Q43, Q44, Q45, Q46, Q47, Q48, Q49, Q5, Q50, Q51, Q52, Q53, Q54, Q55, Q56, Q57, Q58, Q59, Q6, Q60, Q61, Q62, Q63, Q7, Q8, Q9: AO3401A, Package_TO_SOT_SMD:SOT-23, symbol qssc:AO3401A
- removed Re0, Re1, Re10, Re11, Re12, Re13, Re14, Re15, Re16, Re17, Re18, Re19, Re2, Re20, Re21, Re22, Re23, Re24, Re25, Re26, Re27, Re28, Re29, Re3, Re30, Re31, Re32, Re33, Re34, Re35, Re36, Re37, Re38, Re39, Re4, Re40, Re41, Re42, Re43, Re44, Re45, Re46, Re47, Re48, Re49, Re5, Re50, Re51, Re52, Re53, Re54, Re55, Re56, Re57, Re58, Re59, Re6, Re60, Re61, Re62, Re63, Re7, Re8, Re9: 220R, Resistor_SMD:R_0603_1608Metric, symbol qssc:R
- removed Rg0, Rg1, Rg10, Rg11, Rg12, Rg13, Rg14, Rg15, Rg16, Rg17, Rg18, Rg19, Rg2, Rg20, Rg21, Rg22, Rg23, Rg24, Rg25, Rg26, Rg27, Rg28, Rg29, Rg3, Rg30, Rg31, Rg32, Rg33, Rg34, Rg35, Rg36, Rg37, Rg38, Rg39, Rg4, Rg40, Rg41, Rg42, Rg43, Rg44, Rg45, Rg46, Rg47, Rg48, Rg49, Rg5, Rg50, Rg51, Rg52, Rg53, Rg54, Rg55, Rg56, Rg57, Rg58, Rg59, Rg6, Rg60, Rg61, Rg62, Rg63, Rg7, Rg8, Rg9: 100k, Resistor_SMD:R_0603_1608Metric, symbol qssc:R
- removed UB0, UB1, UB2, UB3, UB4, UB5, UB6, UB7: 74HCT240, Package_SO:TSSOP-20_4.4x6.5mm_P0.65mm, symbol qssc:74HCT240
- added C85: 22uF, Capacitor_SMD:C_0805_2012Metric, symbol qssc:C
- added C86, Cem0, Cem1, Cem2: 100nF, Capacitor_SMD:C_0603_1608Metric, symbol qssc:C
- added F2: 1A PTC, Fuse:Fuse_1206_3216Metric, symbol qssc:Polyfuse
- added J4: 12V LED, Connector_BarrelJack:BarrelJack_CUI_PJ-102AH_Horizontal, symbol qssc:Barrel_Jack
- added Riref0, Riref1, Riref2: 4.87k, Resistor_SMD:R_0603_1608Metric, symbol qssc:R
- added UE0, UE1, UE2: TLC5947, Package_SO:HTSSOP-32-1EP_6.1x11mm_P0.65mm_EP5.2x11mm_Mask4.11x4.36mm_ThermalVias, symbol qssc:TLC5947
Connections:
- net EM_DRV11 is gone; now on net DET_DIG54: U1.V15 (DET_DIG54)
- net EM_DRV12 is gone; now on net DET_DIG40: U1.V16 (DET_DIG40)
- net EM_DRV13 is gone; now on net DET_DIG25: U1.V17 (DET_DIG25)
- net EM_DRV26 is gone; now on net DET_DIG39: U1.U16 (DET_DIG39)
- net EM_DRV27 is gone; now on net DET_DIG24: U1.U17 (DET_DIG24)
- net EM_DRV28 is gone; now on net DET_DIG12: U1.U18 (DET_DIG12)
- net EM_DRV40 is gone; now on net DET_DIG53: U1.T15 (DET_DIG53)
- net EM_DRV41 is gone; now on net DET_DIG38: U1.T16 (DET_DIG38)
- net EM_DRV42 is gone; now on net DET_DIG11: U1.T18 (DET_DIG11)
- net EM_DRV54 is gone; now on net DET_DIG52: U1.R15 (DET_DIG52)
- net EM_DRV55 is gone; now on net DET_DIG37: U1.R16 (DET_DIG37)
- net EM_DRV56 is gone; now on net DET_DIG23: U1.R17 (DET_DIG23)
- net EM_DRV57 is gone; now on net DET_DIG10: U1.R18 (DET_DIG10)
- net EM_DRV63 is gone; now on net DET_DIG51: U1.P15 (DET_DIG51)
- net +3V3: now also Cem0.1, Cem1.1, Cem2.1, UE0.32 (VCC), UE1.32 (VCC), UE2.32 (VCC)
- net DET_DIG10: no longer U1.B17 (DET_DIG10)
- net DET_DIG11: no longer U1.C17 (DET_DIG11)
- net DET_DIG12: no longer U1.D17 (DET_DIG12)
- net DET_DIG13: now also U1.B17 (DET_DIG13); no longer U1.E17 (DET_DIG13)
- net DET_DIG14: now also U1.C17 (DET_DIG14); no longer U1.G17 (DET_DIG14)
- net DET_DIG15: now also U1.D17 (DET_DIG15); no longer U1.H17 (DET_DIG15)
- net DET_DIG16: now also U1.E17 (DET_DIG16); no longer U1.J17 (DET_DIG16)
- net DET_DIG17: now also U1.G17 (DET_DIG17); no longer U1.M17 (DET_DIG17)
- net DET_DIG18: now also U1.H17 (DET_DIG18); no longer U1.N17 (DET_DIG18)
- net DET_DIG19: now also U1.J17 (DET_DIG19); no longer U1.P17 (DET_DIG19)
- net DET_DIG20: now also U1.M17 (DET_DIG20); no longer U1.A16 (DET_DIG20)
- net DET_DIG21: now also U1.N17 (DET_DIG21); no longer U1.B16 (DET_DIG21)
- net DET_DIG22: now also U1.P17 (DET_DIG22); no longer U1.C16 (DET_DIG22)
- net DET_DIG23: no longer U1.E16 (DET_DIG23)
- net DET_DIG24: no longer U1.F16 (DET_DIG24)
- net DET_DIG25: no longer U1.G16 (DET_DIG25)
- net DET_DIG26: now also U1.A16 (DET_DIG26); no longer U1.H16 (DET_DIG26)
- net DET_DIG27: now also U1.B16 (DET_DIG27); no longer U1.K16 (DET_DIG27)
- net DET_DIG28: now also U1.C16 (DET_DIG28); no longer U1.L16 (DET_DIG28)
- net DET_DIG29: now also U1.E16 (DET_DIG29); no longer U1.M16 (DET_DIG29)
- net DET_DIG30: now also U1.F16 (DET_DIG30); no longer U1.N16 (DET_DIG30)
- net DET_DIG31: now also U1.G16 (DET_DIG31); no longer U1.A15 (DET_DIG31)
- net DET_DIG32: now also U1.H16 (DET_DIG32); no longer U1.C15 (DET_DIG32)
- net DET_DIG33: now also U1.K16 (DET_DIG33); no longer U1.D15 (DET_DIG33)
- net DET_DIG34: now also U1.L16 (DET_DIG34); no longer U1.E15 (DET_DIG34)
- net DET_DIG35: now also U1.M16 (DET_DIG35); no longer U1.F15 (DET_DIG35)
- net DET_DIG36: now also U1.N16 (DET_DIG36); no longer U1.H15 (DET_DIG36)
- net DET_DIG37: no longer U1.J15 (DET_DIG37)
- net DET_DIG38: no longer U1.K15 (DET_DIG38)
- net DET_DIG39: no longer U1.L15 (DET_DIG39)
- net DET_DIG40: no longer U1.N15 (DET_DIG40)
- net DET_DIG41: now also U1.A15 (DET_DIG41); no longer U1.A14 (DET_DIG41)
- net DET_DIG42: now also U1.C15 (DET_DIG42); no longer U1.B14 (DET_DIG42)
- net DET_DIG43: now also U1.D15 (DET_DIG43); no longer U1.C14 (DET_DIG43)
- net DET_DIG44: now also U1.E15 (DET_DIG44); no longer U1.D14 (DET_DIG44)
- net DET_DIG45: now also U1.F15 (DET_DIG45); no longer U1.F14 (DET_DIG45)
- net DET_DIG46: now also U1.H15 (DET_DIG46); no longer U1.G14 (DET_DIG46)
- net DET_DIG47: now also U1.J15 (DET_DIG47); no longer U1.H14 (DET_DIG47)
- net DET_DIG48: now also U1.K15 (DET_DIG48); no longer U1.J14 (DET_DIG48)
- net DET_DIG49: now also U1.L15 (DET_DIG49); no longer U1.N14 (DET_DIG49)
- net DET_DIG50: now also U1.N15 (DET_DIG50); no longer U1.A13 (DET_DIG50)
- net DET_DIG51: no longer U1.B13 (DET_DIG51)
- net DET_DIG52: no longer U1.D13 (DET_DIG52)
- net DET_DIG53: no longer U1.F13 (DET_DIG53)
- net DET_DIG54: no longer U1.G13 (DET_DIG54)
- net DET_DIG55: now also U1.A14 (DET_DIG55); no longer U1.J13 (DET_DIG55)
- net DET_DIG56: now also U1.B14 (DET_DIG56); no longer U1.K13 (DET_DIG56)
- net DET_DIG57: now also U1.C14 (DET_DIG57); no longer U1.M13 (DET_DIG57)
- net DET_DIG58: now also U1.D14 (DET_DIG58); no longer U1.B12 (DET_DIG58)
- net DET_DIG59: now also U1.F14 (DET_DIG59); no longer U1.C12 (DET_DIG59)
- net DET_DIG60: now also U1.G14 (DET_DIG60); no longer U1.D12 (DET_DIG60)
- net DET_DIG61: now also U1.H14 (DET_DIG61); no longer U1.A11 (DET_DIG61)
- net DET_DIG62: now also U1.J14 (DET_DIG62); no longer U1.B11 (DET_DIG62)
- net DET_DIG63: now also U1.N14 (DET_DIG63); no longer U1.C11 (DET_DIG63)
- net GND: now also C85.2, C86.2, Cem0.2, Cem1.2, Cem2.2, J4.2, Riref0.2, Riref1.2, Riref2.2, UE0.1 (GND), UE0.33 (EP), UE1.1 (GND), UE1.33 (EP), UE2.1 (GND), UE2.33 (EP)
- net EM_DRV0 renamed em_sclk
- net em_sclk: now also UE0.3 (SCLK), UE1.3 (SCLK), UE2.3 (SCLK)
- net EM_DRV1 renamed em_sin
- net em_sin: now also UE0.4 (SIN)
- removed net EM_DRV10: U1.V14 (EM_DRV10)
- removed net EM_DRV14: U1.U1 (EM_DRV14)
- removed net EM_DRV15: U1.U2 (EM_DRV15)
- removed net EM_DRV16: U1.U3 (EM_DRV16)
- removed net EM_DRV17: U1.U4 (EM_DRV17)
- removed net EM_DRV18: U1.U6 (EM_DRV18)
- removed net EM_DRV19: U1.U7 (EM_DRV19)
- net EM_DRV2 renamed em_xlat
- net em_xlat: now also UE0.30 (XLAT), UE1.30 (XLAT), UE2.30 (XLAT)
- removed net EM_DRV20: U1.U8 (EM_DRV20)
- removed net EM_DRV21: U1.U9 (EM_DRV21)
- removed net EM_DRV22: U1.U11 (EM_DRV22)
- removed net EM_DRV23: U1.U12 (EM_DRV23)
- removed net EM_DRV24: U1.U13 (EM_DRV24)
- removed net EM_DRV25: U1.U14 (EM_DRV25)
- removed net EM_DRV29: U1.T1 (EM_DRV29)
- net EM_DRV3 renamed em_blank
- net em_blank: now also UE0.2 (BLANK), UE1.2 (BLANK), UE2.2 (BLANK)
- removed net EM_DRV30: U1.T3 (EM_DRV30)
- removed net EM_DRV31: U1.T4 (EM_DRV31)
- removed net EM_DRV32: U1.T5 (EM_DRV32)
- removed net EM_DRV33: U1.T6 (EM_DRV33)
- removed net EM_DRV34: U1.T8 (EM_DRV34)
- removed net EM_DRV35: U1.T9 (EM_DRV35)
- removed net EM_DRV36: U1.T10 (EM_DRV36)
- removed net EM_DRV37: U1.T11 (EM_DRV37)
- removed net EM_DRV38: U1.T13 (EM_DRV38)
- removed net EM_DRV39: U1.T14 (EM_DRV39)
- removed net EM_DRV4: U1.V6 (EM_DRV4)
- removed net EM_DRV43: U1.R1 (EM_DRV43)
- removed net EM_DRV44: U1.R2 (EM_DRV44)
- removed net EM_DRV45: U1.R3 (EM_DRV45)
- removed net EM_DRV46: U1.R5 (EM_DRV46)
- removed net EM_DRV47: U1.R6 (EM_DRV47)
- removed net EM_DRV48: U1.R7 (EM_DRV48)
- removed net EM_DRV49: U1.R8 (EM_DRV49)
- removed net EM_DRV5: U1.V7 (EM_DRV5)
- removed net EM_DRV50: U1.R10 (EM_DRV50)
- removed net EM_DRV51: U1.R11 (EM_DRV51)
- removed net EM_DRV52: U1.R12 (EM_DRV52)
- removed net EM_DRV53: U1.R13 (EM_DRV53)
- removed net EM_DRV58: U1.P2 (EM_DRV58)
- removed net EM_DRV59: U1.P3 (EM_DRV59)
- removed net EM_DRV6: U1.V9 (EM_DRV6)
- removed net EM_DRV60: U1.P4 (EM_DRV60)
- removed net EM_DRV61: U1.P5 (EM_DRV61)
- removed net EM_DRV62: U1.P14 (EM_DRV62)
- removed net EM_DRV7: U1.V10 (EM_DRV7)
- removed net EM_DRV8: U1.V11 (EM_DRV8)
- removed net EM_DRV9: U1.V12 (EM_DRV9)
- net VREFP renamed +12V_EMIT_IN
- net +12V_EMIT_IN: now also F2.1, J4.1
- net emitter_anode0 renamed emitter_cat0
- net emitter_cat0: now also UE0.5 (OUT0)
- net emitter_anode1 renamed emitter_cat1
- net emitter_cat1: now also UE0.6 (OUT1)
- net emitter_anode10 renamed emitter_cat10
- net emitter_cat10: now also UE0.15 (OUT10)
- net emitter_anode11 renamed emitter_cat11
- net emitter_cat11: now also UE0.16 (OUT11)
- net emitter_anode12 renamed emitter_cat12
- net emitter_cat12: now also UE0.17 (OUT12)
- net emitter_anode13 renamed emitter_cat13
- net emitter_cat13: now also UE0.18 (OUT13)
- net emitter_anode14 renamed emitter_cat14
- net emitter_cat14: now also UE0.19 (OUT14)
- net emitter_anode15 renamed emitter_cat15
- net emitter_cat15: now also UE0.20 (OUT15)
- net emitter_anode16 renamed emitter_cat16
- net emitter_cat16: now also UE0.21 (OUT16)
- net emitter_anode17 renamed emitter_cat17
- net emitter_cat17: now also UE0.22 (OUT17)
- net emitter_anode18 renamed emitter_cat18
- net emitter_cat18: now also UE0.23 (OUT18)
- net emitter_anode19 renamed emitter_cat19
- net emitter_cat19: now also UE0.24 (OUT19)
- net emitter_anode2 renamed emitter_cat2
- net emitter_cat2: now also UE0.7 (OUT2)
- net emitter_anode20 renamed emitter_cat20
- net emitter_cat20: now also UE0.25 (OUT20)
- net emitter_anode21 renamed emitter_cat21
- net emitter_cat21: now also UE0.26 (OUT21)
- net emitter_anode22 renamed emitter_cat22
- net emitter_cat22: now also UE0.27 (OUT22)
- net emitter_anode23 renamed emitter_cat23
- net emitter_cat23: now also UE0.28 (OUT23)
- net emitter_anode24 renamed emitter_cat24
- net emitter_cat24: now also UE1.5 (OUT0)
- net emitter_anode25 renamed emitter_cat25
- net emitter_cat25: now also UE1.6 (OUT1)
- net emitter_anode26 renamed emitter_cat26
- net emitter_cat26: now also UE1.7 (OUT2)
- net emitter_anode27 renamed emitter_cat27
- net emitter_cat27: now also UE1.8 (OUT3)
- net emitter_anode28 renamed emitter_cat28
- net emitter_cat28: now also UE1.9 (OUT4)
- net emitter_anode29 renamed emitter_cat29
- net emitter_cat29: now also UE1.10 (OUT5)
- net emitter_anode3 renamed emitter_cat3
- net emitter_cat3: now also UE0.8 (OUT3)
- net emitter_anode30 renamed emitter_cat30
- net emitter_cat30: now also UE1.11 (OUT6)
- net emitter_anode31 renamed emitter_cat31
- net emitter_cat31: now also UE1.12 (OUT7)
- net emitter_anode32 renamed emitter_cat32
- net emitter_cat32: now also UE1.13 (OUT8)
- net emitter_anode33 renamed emitter_cat33
- net emitter_cat33: now also UE1.14 (OUT9)
- net emitter_anode34 renamed emitter_cat34
- net emitter_cat34: now also UE1.15 (OUT10)
- net emitter_anode35 renamed emitter_cat35
- net emitter_cat35: now also UE1.16 (OUT11)
- net emitter_anode36 renamed emitter_cat36
- net emitter_cat36: now also UE1.17 (OUT12)
- net emitter_anode37 renamed emitter_cat37
- net emitter_cat37: now also UE1.18 (OUT13)
- net emitter_anode38 renamed emitter_cat38
- net emitter_cat38: now also UE1.19 (OUT14)
- net emitter_anode39 renamed emitter_cat39
- net emitter_cat39: now also UE1.20 (OUT15)
- net emitter_anode4 renamed emitter_cat4
- net emitter_cat4: now also UE0.9 (OUT4)
- net emitter_anode40 renamed emitter_cat40
- net emitter_cat40: now also UE1.21 (OUT16)
- net emitter_anode41 renamed emitter_cat41
- net emitter_cat41: now also UE1.22 (OUT17)
- net emitter_anode42 renamed emitter_cat42
- net emitter_cat42: now also UE1.23 (OUT18)
- net emitter_anode43 renamed emitter_cat43
- net emitter_cat43: now also UE1.24 (OUT19)
- net emitter_anode44 renamed emitter_cat44
- net emitter_cat44: now also UE1.25 (OUT20)
- net emitter_anode45 renamed emitter_cat45
- net emitter_cat45: now also UE1.26 (OUT21)
- net emitter_anode46 renamed emitter_cat46
- net emitter_cat46: now also UE1.27 (OUT22)
- net emitter_anode47 renamed emitter_cat47
- net emitter_cat47: now also UE1.28 (OUT23)
- net emitter_anode48 renamed emitter_cat48
- net emitter_cat48: now also UE2.5 (OUT0)
- net emitter_anode49 renamed emitter_cat49
- net emitter_cat49: now also UE2.6 (OUT1)
- net emitter_anode5 renamed emitter_cat5
- net emitter_cat5: now also UE0.10 (OUT5)
- net emitter_anode50 renamed emitter_cat50
- net emitter_cat50: now also UE2.7 (OUT2)
- net emitter_anode51 renamed emitter_cat51
- net emitter_cat51: now also UE2.8 (OUT3)
- net emitter_anode52 renamed emitter_cat52
- net emitter_cat52: now also UE2.9 (OUT4)
- net emitter_anode53 renamed emitter_cat53
- net emitter_cat53: now also UE2.10 (OUT5)
- net emitter_anode54 renamed emitter_cat54
- net emitter_cat54: now also UE2.11 (OUT6)
- net emitter_anode55 renamed emitter_cat55
- net emitter_cat55: now also UE2.12 (OUT7)
- net emitter_anode56 renamed emitter_cat56
- net emitter_cat56: now also UE2.13 (OUT8)
- net emitter_anode57 renamed emitter_cat57
- net emitter_cat57: now also UE2.14 (OUT9)
- net emitter_anode58 renamed emitter_cat58
- net emitter_cat58: now also UE2.15 (OUT10)
- net emitter_anode59 renamed emitter_cat59
- net emitter_cat59: now also UE2.16 (OUT11)
- net emitter_anode6 renamed emitter_cat6
- net emitter_cat6: now also UE0.11 (OUT6)
- net emitter_anode60 renamed emitter_cat60
- net emitter_cat60: now also UE2.17 (OUT12)
- net emitter_anode61 renamed emitter_cat61
- net emitter_cat61: now also UE2.18 (OUT13)
- net emitter_anode62 renamed emitter_cat62
- net emitter_cat62: now also UE2.19 (OUT14)
- net emitter_anode63 renamed emitter_cat63
- net emitter_cat63: now also UE2.20 (OUT15)
- net emitter_anode7 renamed emitter_cat7
- net emitter_cat7: now also UE0.12 (OUT7)
- net emitter_anode8 renamed emitter_cat8
- net emitter_cat8: now also UE0.13 (OUT8)
- net emitter_anode9 renamed emitter_cat9
- net emitter_cat9: now also UE0.14 (OUT9)
- new net +12V_EMIT: C85.1, C86.1, F2.2, Uchip.EM_ANODE
- new net em_iref0: Riref0.1, UE0.31 (IREF)
- new net em_iref1: Riref1.1, UE1.31 (IREF)
- new net em_iref2: Riref2.1, UE2.31 (IREF)
- new net em_sout0: UE0.29 (SOUT), UE1.4 (SIN)
- new net em_sout1: UE1.29 (SOUT), UE2.4 (SIN)

Commit message: pcb: two-board sandwich routed + DRC/ERC 0/0, HDI via rules
Split the single merged board into the production two-PCB sandwich for the
two-faced (no-TSV) QSSC die:

- Main board (qssc, 6-layer 210x140): FPGA + 3x TLC5947 emitter + RF + USB +
  power, die BOTTOM/emitter face on F.Cu (ACF pressure contact), BTB HOST J12.
- Detector head (chip_module, 4-layer 150x140): 16x TLV9004 TIA + 4x AD7616
  ADC, die TOP/detector face on B.Cu+B.Mask (no B.Paste), BTB DAUGHTER J12.
  Head origin = main origin + (60,0)mm so J12 and die footprints align.
- BTB J12 carries the 9-wire AD7616 SPI + GND/+3V3/+5V; identical net names
  on both boards. RTL and Qiskit software unchanged.

Generator (gen_qssc_kicad.py): parameterized emit_schematic/emit_pcb/emit_pro
on a per-board cfg; HEAD_LAYER_STACK/HEAD_STACK_UP/HEAD_CFG + build_detector_head
+ assign_pcb_positions_head; split chip face into QSSC_Chip_EM (F.Cu) /
QSSC_Chip_DET (B.Cu); authored Conn_02x10_BTB; main() emits both boards.
emit_pro design rules now match the HDI stackup: min_via_diameter 0.45->0.20,
min_via_annular_width 0.10->0.05 (agrees with route_signals
_relax_board_for_hdi: 0.20 mm VIP / 0.05 mm via-in-pad annular). The old
0.45/0.10 floor flagged every routing (0.40 mm) and BGA dog-bone (0.20 mm)
via as via_diameter/annular_width.

Router (route_signals.py): SIGNAL/PLANE/JUMP layers recomputed from
GetCopperLayerCount (4-layer head safe); _chip_fanout stub/escape derived
from the pad's own layer (DET pads escape on F.Cu, EM pads on B.Cu); _FpProxy
stores x,y so the snapshot proxy has a position.

Result (fresh gen -> route_signals -> route_qssc_pcb -> kicad-cli):
  qssc        DRC 0 violations, ERC 0 errors
  chip_module DRC 0 violations, ERC 0 errors
Main: 26/130 nets 1st-pass + 2 planes (GND/+3V3) + 398 vias; 100 unrouted
(64 emitter cathodes + FPGA config/RF/USB) left for FreeRouting.
Head: 10/156 nets 1st-pass + 2 planes + 435 vias; 146 unrouted (DET->TIA->
ADC analog + SPI) left for FreeRouting.

Co-Authored-By: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
Parts:
- removed Cdac, Cref, Cuc0, Cuc1, Cuc10, Cuc11, Cuc12, Cuc13, Cuc14, Cuc15, Cuc2, Cuc3, Cuc4, Cuc5, Cuc6, Cuc7, Cuc8, Cuc9, Cut0, Cut1, Cut10, Cut11, Cut12, Cut13, Cut14, Cut15, Cut2, Cut3, Cut4, Cut5, Cut6, Cut7, Cut8, Cut9: 100nF, Capacitor_SMD:C_0603_1608Metric, symbol qssc:C
- removed Cf0, Cf1, Cf10, Cf11, Cf12, Cf13, Cf14, Cf15, Cf16, Cf17, Cf18, Cf19, Cf2, Cf20, Cf21, Cf22, Cf23, Cf24, Cf25, Cf26, Cf27, Cf28, Cf29, Cf3, Cf30, Cf31, Cf32, Cf33, Cf34, Cf35, Cf36, Cf37, Cf38, Cf39, Cf4, Cf40, Cf41, Cf42, Cf43, Cf44, Cf45, Cf46, Cf47, Cf48, Cf49, Cf5, Cf50, Cf51, Cf52, Cf53, Cf54, Cf55, Cf56, Cf57, Cf58, Cf59, Cf6, Cf60, Cf61, Cf62, Cf63, Cf7, Cf8, Cf9: 1pF, Capacitor_SMD:C_0603_1608Metric, symbol qssc:C
- removed R_I2C_SCL, R_I2C_SDA: 4.7k, Resistor_SMD:R_0603_1608Metric, symbol qssc:R
- removed Rf0, Rf1, Rf10, Rf11, Rf12, Rf13, Rf14, Rf15, Rf16, Rf17, Rf18, Rf19, Rf2, Rf20, Rf21, Rf22, Rf23, Rf24, Rf25, Rf26, Rf27, Rf28, Rf29, Rf3, Rf30, Rf31, Rf32, Rf33, Rf34, Rf35, Rf36, Rf37, Rf38, Rf39, Rf4, Rf40, Rf41, Rf42, Rf43, Rf44, Rf45, Rf46, Rf47, Rf48, Rf49, Rf5, Rf50, Rf51, Rf52, Rf53, Rf54, Rf55, Rf56, Rf57, Rf58, Rf59, Rf6, Rf60, Rf61, Rf62, Rf63, Rf7, Rf8, Rf9: 1M, Resistor_SMD:R_0603_1608Metric, symbol qssc:R
- removed Rpu0, Rpu1, Rpu10, Rpu11, Rpu12, Rpu13, Rpu14, Rpu15, Rpu16, Rpu17, Rpu18, Rpu19, Rpu2, Rpu20, Rpu21, Rpu22, Rpu23, Rpu24, Rpu25, Rpu26, Rpu27, Rpu28, Rpu29, Rpu3, Rpu30, Rpu31, Rpu32, Rpu33, Rpu34, Rpu35, Rpu36, Rpu37, Rpu38, Rpu39, Rpu4, Rpu40, Rpu41, Rpu42, Rpu43, Rpu44, Rpu45, Rpu46, Rpu47, Rpu48, Rpu49, Rpu5, Rpu50, Rpu51, Rpu52, Rpu53, Rpu54, Rpu55, Rpu56, Rpu57, Rpu58, Rpu59, Rpu6, Rpu60, Rpu61, Rpu62, Rpu63, Rpu7, Rpu8, Rpu9, Rref1, Rref2: 10k, Resistor_SMD:R_0603_1608Metric, symbol qssc:R
- removed UC0, UC1, UC10, UC11, UC12, UC13, UC14, UC15, UC2, UC3, UC4, UC5, UC6, UC7, UC8, UC9: LMV339, Package_SO:SOIC-14_3.9x8.7mm_P1.27mm, symbol qssc:LMV339
- removed UDAC: MCP4725, Package_TO_SOT_SMD:SOT-23-6, symbol qssc:MCP4725
- removed UT0, UT1, UT10, UT11, UT12, UT13, UT14, UT15, UT2, UT3, UT4, UT5, UT6, UT7, UT8, UT9: TLV9004, Package_SO:TSSOP-14_4.4x5mm_P0.65mm, symbol qssc:TLV9004
- removed Uchip: QSSC_Chip, qssc:QSSC_Chip, symbol qssc:QSSC_Chip
- added J12: BTB_HOST, qssc:Conn_02x10_BTB, symbol qssc:Conn_02x10_BTB
- added Uchip: QSSC_Chip_EM, qssc:QSSC_Chip_EM, symbol qssc:QSSC_Chip_EM
Connections:
- net +12V_EMIT: now also Uchip.EM_ANODE
- net +12V_EMIT_IN: no longer C40.1, U1.K10 (VREFP)
- net +3V3: now also J12.2
- net +5V: now also J12.17, J12.18
- net GND: now also J12.1, J12.10, J12.12, J12.19, J12.20, J12.4, J12.6, J12.8
- net emitter_cat0: now also Uchip.EM0
- net emitter_cat1: now also Uchip.EM1
- net emitter_cat10: now also Uchip.EM10
- net emitter_cat11: now also Uchip.EM11
- net emitter_cat12: now also Uchip.EM12
- net emitter_cat13: now also Uchip.EM13
- net emitter_cat14: now also Uchip.EM14
- net emitter_cat15: now also Uchip.EM15
- net emitter_cat16: now also Uchip.EM16
- net emitter_cat17: now also Uchip.EM17
- net emitter_cat18: now also Uchip.EM18
- net emitter_cat19: now also Uchip.EM19
- net emitter_cat2: now also Uchip.EM2
- net emitter_cat20: now also Uchip.EM20
- net emitter_cat21: now also Uchip.EM21
- net emitter_cat22: now also Uchip.EM22
- net emitter_cat23: now also Uchip.EM23
- net emitter_cat24: now also Uchip.EM24
- net emitter_cat25: now also Uchip.EM25
- net emitter_cat26: now also Uchip.EM26
- net emitter_cat27: now also Uchip.EM27
- net emitter_cat28: now also Uchip.EM28
- net emitter_cat29: now also Uchip.EM29
- net emitter_cat3: now also Uchip.EM3
- net emitter_cat30: now also Uchip.EM30
- net emitter_cat31: now also Uchip.EM31
- net emitter_cat32: now also Uchip.EM32
- net emitter_cat33: now also Uchip.EM33
- net emitter_cat34: now also Uchip.EM34
- net emitter_cat35: now also Uchip.EM35
- net emitter_cat36: now also Uchip.EM36
- net emitter_cat37: now also Uchip.EM37
- net emitter_cat38: now also Uchip.EM38
- net emitter_cat39: now also Uchip.EM39
- net emitter_cat4: now also Uchip.EM4
- net emitter_cat40: now also Uchip.EM40
- net emitter_cat41: now also Uchip.EM41
- net emitter_cat42: now also Uchip.EM42
- net emitter_cat43: now also Uchip.EM43
- net emitter_cat44: now also Uchip.EM44
- net emitter_cat45: now also Uchip.EM45
- net emitter_cat46: now also Uchip.EM46
- net emitter_cat47: now also Uchip.EM47
- net emitter_cat48: now also Uchip.EM48
- net emitter_cat49: now also Uchip.EM49
- net emitter_cat5: now also Uchip.EM5
- net emitter_cat50: now also Uchip.EM50
- net emitter_cat51: now also Uchip.EM51
- net emitter_cat52: now also Uchip.EM52
- net emitter_cat53: now also Uchip.EM53
- net emitter_cat54: now also Uchip.EM54
- net emitter_cat55: now also Uchip.EM55
- net emitter_cat56: now also Uchip.EM56
- net emitter_cat57: now also Uchip.EM57
- net emitter_cat58: now also Uchip.EM58
- net emitter_cat59: now also Uchip.EM59
- net emitter_cat6: now also Uchip.EM6
- net emitter_cat60: now also Uchip.EM60
- net emitter_cat61: now also Uchip.EM61
- net emitter_cat62: now also Uchip.EM62
- net emitter_cat63: now also Uchip.EM63
- net emitter_cat7: now also Uchip.EM7
- net emitter_cat8: now also Uchip.EM8
- net emitter_cat9: now also Uchip.EM9
- net DET_DIG0 renamed adc_convst
- net adc_convst: now also J12.3
- net DET_DIG1 renamed adc_sclk
- net adc_sclk: now also J12.5
- removed net DET_DIG10: U1.R18 (DET_DIG10)
- removed net DET_DIG11: U1.T18 (DET_DIG11)
- removed net DET_DIG12: U1.U18 (DET_DIG12)
- removed net DET_DIG13: U1.B17 (DET_DIG13)
- removed net DET_DIG14: U1.C17 (DET_DIG14)
- removed net DET_DIG15: U1.D17 (DET_DIG15)
- removed net DET_DIG16: U1.E17 (DET_DIG16)
- removed net DET_DIG17: U1.G17 (DET_DIG17)
- removed net DET_DIG18: U1.H17 (DET_DIG18)
- removed net DET_DIG19: U1.J17 (DET_DIG19)
- net DET_DIG2 renamed adc_miso
- net adc_miso: now also J12.7
- removed net DET_DIG20: U1.M17 (DET_DIG20)
- removed net DET_DIG21: U1.N17 (DET_DIG21)
- removed net DET_DIG22: U1.P17 (DET_DIG22)
- removed net DET_DIG23: U1.R17 (DET_DIG23)
- removed net DET_DIG24: U1.U17 (DET_DIG24)
- removed net DET_DIG25: U1.V17 (DET_DIG25)
- removed net DET_DIG26: U1.A16 (DET_DIG26)
- removed net DET_DIG27: U1.B16 (DET_DIG27)
- removed net DET_DIG28: U1.C16 (DET_DIG28)
- removed net DET_DIG29: U1.E16 (DET_DIG29)
- net DET_DIG3 renamed adc_busy
- net adc_busy: now also J12.9
- removed net DET_DIG30: U1.F16 (DET_DIG30)
- removed net DET_DIG31: U1.G16 (DET_DIG31)
- removed net DET_DIG32: U1.H16 (DET_DIG32)
- removed net DET_DIG33: U1.K16 (DET_DIG33)
- removed net DET_DIG34: U1.L16 (DET_DIG34)
- removed net DET_DIG35: U1.M16 (DET_DIG35)
- removed net DET_DIG36: U1.N16 (DET_DIG36)
- removed net DET_DIG37: U1.R16 (DET_DIG37)
- removed net DET_DIG38: U1.T16 (DET_DIG38)
- removed net DET_DIG39: U1.U16 (DET_DIG39)
- net DET_DIG4 renamed adc_cs0
- net adc_cs0: now also J12.13
- removed net DET_DIG40: U1.V16 (DET_DIG40)
- removed net DET_DIG41: U1.A15 (DET_DIG41)
- removed net DET_DIG42: U1.C15 (DET_DIG42)
- removed net DET_DIG43: U1.D15 (DET_DIG43)
- removed net DET_DIG44: U1.E15 (DET_DIG44)
- removed net DET_DIG45: U1.F15 (DET_DIG45)
- removed net DET_DIG46: U1.H15 (DET_DIG46)
- removed net DET_DIG47: U1.J15 (DET_DIG47)
- removed net DET_DIG48: U1.K15 (DET_DIG48)
- removed net DET_DIG49: U1.L15 (DET_DIG49)
- net DET_DIG5 renamed adc_cs1
- net adc_cs1: now also J12.14
- removed net DET_DIG50: U1.N15 (DET_DIG50)
- removed net DET_DIG51: U1.P15 (DET_DIG51)
- removed net DET_DIG52: U1.R15 (DET_DIG52)
- removed net DET_DIG53: U1.T15 (DET_DIG53)
- removed net DET_DIG54: U1.V15 (DET_DIG54)
- removed net DET_DIG55: U1.A14 (DET_DIG55)
- removed net DET_DIG56: U1.B14 (DET_DIG56)
- removed net DET_DIG57: U1.C14 (DET_DIG57)
- removed net DET_DIG58: U1.D14 (DET_DIG58)
- removed net DET_DIG59: U1.F14 (DET_DIG59)
- net DET_DIG6 renamed adc_cs2
- net adc_cs2: now also J12.15
- removed net DET_DIG60: U1.G14 (DET_DIG60)
- removed net DET_DIG61: U1.H14 (DET_DIG61)
- removed net DET_DIG62: U1.J14 (DET_DIG62)
- removed net DET_DIG63: U1.N14 (DET_DIG63)
- net DET_DIG7 renamed adc_cs3
- net adc_cs3: now also J12.16
- net DET_DIG8 renamed adc_resetn
- net adc_resetn: now also J12.11
- removed net DET_DIG9: U1.P18 (DET_DIG9)
- removed net I2C_SCL: U1.N1 (I2C_SCL)
- removed net I2C_SDA: U1.M1 (I2C_SDA)
- new net VREFP: C40.1, U1.K10 (VREFP)
Other:
- title: QSSC Control Board -> QSSC Main Control Board
