File: hardware/pcb/qssc.kicad_pcb (KiCad board)
At the start: 6 copper layers, 210 x 140 mm, 126 parts, among them J1 FT232RL, J10 USB-C, J12 BTB_HOST, J2 5V Barrel, J3 SMA, J4 12V LED, J7 RESET, J8 MW_GATE, J9 JTAG, U1 XC7A35T-1CSG324C, U3 ADF4351BCPZ, U5 GVA-84+, U8 W25Q128JVSIQ, Y1 100MHz XO

Commit message: latest boards 2 pcb first route
Routing:
- net ADF_TEMP: track 0.85 -> 11.0 mm, vias 1 -> 2
- net LF_OUT: track 16.7 -> 20.6 mm, vias 2 -> 3
- net TCK: track 154.6 -> 153.4 mm
