File: hardware/pcb/qssc-grad.kicad_sch (KiCad schematic)
At the start: 133 parts, among them J1 FT232RL, J10 USB-C, J12 BTB_HOST, J2 5V Barrel, J3 SMA, J4 12V LED, J7 RESET, J8 MW_GATE, J9 JTAG, U1 XC7A35T-1CSG324C, U3 ADF4351BCPZ, U5 GVA-84+, U8 W25Q128JVSIQ, Y1 100MHz XO

Commit message: pcb: qssc-grad net-tie coil + Rgrad_feed + V-row grad pins — DRC 0/0/0
Fixes the Invention-5 gradient coil blockers found in the variant review:

1. Coil is now a real KiCad net-tie footprint (net_tie_pad_groups "1, 2")
   with a filled fp_poly on F.Cu -- the coil trace CONDUCTS (was F.Fab =
   open circuit).  A 0R feed resistor Rgrad_feed bridges +5V -> GRAD_COIL_P
   -> Lgrad pad1, so the +5V plane and GRAD_COIL_N stay separate everywhere
   except at the resistor: the MOSFET drain cannot bypass the coil via the
   +5V plane.  Lgrad pad1 = GRAD_COIL_P, pad2 = GRAD_COIL_N.

2. grad FPGA pins moved to the south edge (V6/V9/V12/V7) in xdc + ballmap +
   generator net map -- the old M1/N1/R1/T1 pins conflicted with base-board
   inner-layer escapes.  grad_sclk (V9) gets a pre-placed dogbone fanout via
   (add_grad_fanout) so the 3D maze router can escape the BGA.

3. maze_bridge_3d.py de-forked: --keep-power[=NET,..] flag replaces the
   separate maze_bridge_3d_pwr.py (deleted).  Routes all 10 grad nets + the
   +5V feed across B.Cu/In3/In4/F.Cu with via transitions.

4. Generator min_hole_to_hole 0.25 -> 0.20 to match the hand-routed main
   board (whose dense 0.10mm-drill HDI vias were DRC'd at 0.20); the old
   0.25 tripped 3 hole_near_hole errors on re-injected emitter_cat vias.

5. Deleted stale tools: fix_uchip_pads.py (wrong premise -- main board uses
   the 1.7mm PTH female-header socket, not 1.2mm SMD ACF) + maze_bridge_3d_pwr.py
   + tracked chip_module.closed.* scratch boards.

Result: qssc-grad 2448 tracks / 817 vias, DRC 0 errors / 0 unconnected / 0
footprint errors, ERC 0.  Base qssc.*/chip_module.* boards byte-unchanged.

Co-Authored-By: Claude Code <noreply@anthropic.com>
Parts:
- added Rgrad_feed: 0R, Resistor_SMD:R_0805_2012Metric, symbol qssc:R
Connections:
- net +5V: now also Rgrad_feed.1; no longer Lgrad.1
- net grad_cs: now also U1.V6 (grad_cs); no longer U1.M1 (grad_cs)
- net grad_en: now also U1.V7 (grad_en); no longer U1.T1 (grad_en)
- net grad_mosi: now also U1.V12 (grad_mosi); no longer U1.R1 (grad_mosi)
- net grad_sclk: now also U1.V9 (grad_sclk); no longer U1.N1 (grad_sclk)
- new net GRAD_COIL_P: Lgrad.1, Rgrad_feed.2
Changed lines of the file:
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@@
 		(pin "L14"
 		)
-		(pin "M1"
-		)
 		(pin "M14"
 		)
-		(pin "N1"
-		)
 		(pin "P10"
 		)
-		(pin "R1"
-		)
-		(pin "T1"
-		)
 		(pin "V1"
 		)
+		(pin "V12"
+		)
 		(pin "V2"
 		)
@@
 		(pin "V5"
 		)
+		(pin "V6"
+		)
+		(pin "V7"
+		)
+		(pin "V9"
+		)
 		(pin "A17"
 		)
@@
 	)
 	(symbol
-		(lib_id "qssc:L")
+		(lib_id "qssc:R")
 		(at 684.0 20.0 0)
 		(unit 1)
@@
 		(on_board yes)
 		(dnp no)
-		(property "Reference" "Lgrad"
+		(property "Reference" "Rgrad_feed"
 			(at 684.0 18.0 0)
 			(effects
@@
 			)
 		)
-		(property "Value" "GradCoil"
+		(property "Value" "0R"
 			(at 684.0 22.0 0)
 			(effects
@@
 			)
 		)
-		(property "Footprint" "qssc:GradCoil"
+		(property "Footprint" "Resistor_SMD:R_0805_2012Metric"
 			(at 684.0 20.0 0)
 			(effects
@@
 			(project "qssc-grad"
 				(path "/00000000-0000-0000-0000-000000000001"
-					(reference "Lgrad")
+					(reference "Rgrad_feed")
 					(unit 1)
 				)
@@
 	)
 	(symbol
-		(lib_id "qssc:R")
+		(lib_id "qssc:L")
 		(at 706.0 20.0 0)
 		(unit 1)
@@
 		(on_board yes)
 		(dnp no)
-		(property "Reference" "Rsense"
+		(property "Reference" "Lgrad"
 			(at 706.0 18.0 0)
 			(effects
@@
 			)
 		)
-		(property "Value" "1"
+		(property "Value" "GradCoil"
 			(at 706.0 22.0 0)
 			(effects
@@
 			)
 		)
-		(property "Footprint" "Resistor_SMD:R_2512_6332Metric"
+		(property "Footprint" "qssc:GradCoil"
 			(at 706.0 20.0 0)
 			(effects
@@
 			(project "qssc-grad"
 				(path "/00000000-0000-0000-0000-000000000001"
-					(reference "Rsense")
+					(reference "Lgrad")
 					(unit 1)
 				)
@@
 	)
 	(symbol
-		(lib_id "qssc:C")
+		(lib_id "qssc:R")
 		(at 728.0 20.0 0)
 		(unit 1)
@@
 		(on_board yes)
 		(dnp no)
-		(property "Reference" "C_grad1"
+		(property "Reference" "Rsense"
 			(at 728.0 18.0 0)
 			(effects
@@
 			)
 		)
-		(property "Value" "100nF"
+		(property "Value" "1"
 			(at 728.0 22.0 0)
 			(effects
@@
 			)
 		)
-		(property "Footprint" "Capacitor_SMD:C_0603_1608Metric"
+		(property "Footprint" "Resistor_SMD:R_2512_6332Metric"
 			(at 728.0 20.0 0)
 			(effects
@@
 			(project "qssc-grad"
 				(path "/00000000-0000-0000-0000-000000000001"
-					(reference "C_grad1")
+					(reference "Rsense")
 					(unit 1)
 				)
@@
 		(on_board yes)
 		(dnp no)
-		(property "Reference" "C_grad2"
+		(property "Reference" "C_grad1"
 			(at 750.0 18.0 0)
 			(effects
@@
 			(project "qssc-grad"
 				(path "/00000000-0000-0000-0000-000000000001"
+					(reference "C_grad1")
+					(unit 1)
+				)
+			)
+		)
+	)
+	(symbol
+		(lib_id "qssc:C")
+		(at 772.0 20.0 0)
+		(unit 1)
+		(exclude_from_sim no)
+		(in_bom yes)
+		(on_board yes)
+		(dnp no)
+		(property "Reference" "C_grad2"
+			(at 772.0 18.0 0)
+			(effects
+				(font
+					(size 1.27 1.27)
+				)
+			)
+		)
+		(property "Value" "100nF"
+			(at 772.0 22.0 0)
+			(effects
+				(font
+					(size 1.27 1.27)
+				)
+			)
+		)
+		(property "Footprint" "Capacitor_SMD:C_0603_1608Metric"
+			(at 772.0 20.0 0)
+			(effects
+				(font
+					(size 1.27 1.27)
+				)
+				(hide yes)
+			)
+		)
+		(pin "1"
+		)
+		(pin "2"
+		)
+		(instances
+			(project "qssc-grad"
+				(path "/00000000-0000-0000-0000-000000000001"
 					(reference "C_grad2")
 					(unit 1)
@@
 	)
 	(label "em_blank"
-		(at 250.8 83.97 0)
+		(at 250.8 80.16 0)
 		(fields_autoplaced yes)
 		(effects
@@
 	)
 	(label "em_sclk"
-		(at 250.8 80.16 0)
+		(at 250.8 75.08 0)
 		(fields_autoplaced yes)
 		(effects
@@
 	)
 	(label "em_sin"
-		(at 250.8 81.43 0)
+		(at 250.8 77.62 0)
 		(fields_autoplaced yes)
 		(effects
@@
 	)
 	(label "em_xlat"
-		(at 250.8 82.7 0)
+		(at 250.8 78.89 0)
 		(fields_autoplaced yes)
 		(effects
@@
 	)
 	(label "grad_cs"
-		(at 250.8 72.54 0)
+		(at 250.8 81.43 0)
 		(fields_autoplaced yes)
 		(effects
@@
 	)
 	(label "grad_en"
-		(at 250.8 78.89 0)
+		(at 250.8 82.7 0)
 		(fields_autoplaced yes)
 		(effects
@@
 	)
 	(label "grad_mosi"
-		(at 250.8 77.62 0)
+		(at 250.8 76.35 0)
 		(fields_autoplaced yes)
 		(effects
@@
 	)
 	(label "grad_sclk"
-		(at 250.8 75.08 0)
+		(at 250.8 83.97 0)
 		(fields_autoplaced yes)
 		(effects
@@
 	)
 	(label "SPI_D3"
-		(at 250.8 73.81 0)
+		(at 250.8 72.54 0)
 		(fields_autoplaced yes)
 		(effects
@@
 	)
 	(label "CONF_DONE"
-		(at 250.8 76.35 0)
+		(at 250.8 73.81 0)
 		(fields_autoplaced yes)
 		(effects
@@
 		)
 	)
-	(label "GRAD_COIL_N"
+	(label "GRAD_COIL_P"
 		(at 684.0 23.81 0)
 		(fields_autoplaced yes)
@@
 		)
 	)
-	(label "GRAD_SENSE"
+	(label "GRAD_COIL_P"
 		(at 706.0 16.19 0)
 		(fields_autoplaced yes)
@@
 		)
 	)
-	(label "GND"
+	(label "GRAD_COIL_N"
 		(at 706.0 23.81 0)
 		(fields_autoplaced yes)
@@
 		)
 	)
-	(label "+5V"
+	(label "GRAD_SENSE"
 		(at 728.0 16.19 0)
 		(fields_autoplaced yes)
@@
 		(fields_autoplaced yes)
 		(effects
+			(font
+				(size 1.27 1.27)
+			)
+			(justify left bottom)
+		)
+	)
+	(label "+5V"
+		(at 772.0 16.19 0)
+		(fields_autoplaced yes)
+		(effects
+			(font
+				(size 1.27 1.27)
+			)
+			(justify left bottom)
+		)
+	)
+	(label "GND"
+		(at 772.0 23.81 0)
+		(fields_autoplaced yes)
+		(effects
