File: hardware/pcb/qssc-grad.kicad_pcb (KiCad board)
At the start: 6 copper layers, 150 x 118 mm, 134 parts, among them J1 FT232RL, J10 USB-C, J12 BTB_HOST, J2 5V Barrel, J3 SMA, J4 12V LED, J7 RESET, J8 MW_GATE, J9 JTAG, U1 XC7A35T-1CSG324C, U3 ADF4351BCPZ, U5 GVA-84+, U8 W25Q128JVSIQ, Y1 100MHz XO

Commit message: fix(hardware): LM358 V-/V+ swap, MPN repairs, full grad copper repair, gate re-pins
- LM358 library symbol pins: 4 VCC->V-, 8 GND->V+ (real LM358 pinout)
- grad SCH: +5V/GND labels swapped at the UDRV pins; board pads swapped to
  match (Udrv pad 4 = GND, pad 8 = +5V); schematic_parity 0 in kicad-cli DRC
- BOM: J9 61300411121 -> 61301011121 (2x05 needs 10 contacts), Udrv
  LM358P -> LM358DR; the BOM delta pin (test_dumb_mistakes) re-pinned to
  exactly the reviewed 2 removes / 3 adds (issues #168/#169)
- grad PCB: all 12 formerly stranded cluster pads routed (net 6 +5V: 12
  F.Cu segments incl. the Rgrad_feed west route and the north-edge bridge
  to the existing +5V via at (114.04, 5.11); net 18 GND: 15 F.Cu segments;
  net 24 GRAD_SENSE: 2). No new via: the planned through-via at (139.5,
  94.8) was retracted after a ray-cast point-in-polygon check showed it
  inside the committed In1 (GND) and In2 (+3V3) pours -- the F.Cu-only
  bridge keeps both inner planes intact, no zone refill needed.
- electrical sanity: the four repaired gates re-pinned green (markers
  dropped); the MCP4921 VDD xfail stays (defect 3 open)
- DRC (kicad-cli): 0 violations, 0 unconnected, 0 schematic parity; full
  suite captures show exactly one failing test (known pre-existing C87
  placement, test_bom_matches_board[main]) and no unexpected XPASS

[skip ci]

Co-Authored-By: Claude <noreply@anthropic.com>
Connections:
- Udrv pad 4: +5V -> GND
- Udrv pad 8: GND -> +5V
Routing:
- net +5V: track 247.0 -> 497.6 mm
- net GND: track 71.8 -> 110.8 mm
- net GRAD_SENSE: track 9.91 -> 21.0 mm
Changed lines of the file:
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@@
 			(layers "F.Cu" "F.Paste" "F.Mask")
 			(roundrect_rratio 0.25)
-			(net 6 "+5V")
+			(net 18 "GND")
 		)
 		(pad "5" smd roundrect
@@
 			(layers "F.Cu" "F.Paste" "F.Mask")
 			(roundrect_rratio 0.25)
-			(net 18 "GND")
+			(net 6 "+5V")
 		)
 		(model "${KICAD8_3DMODEL_DIR}/Package_SO.3dshapes/SOIC-8_3.9x4.9mm_P1.27mm.wrl"
@@
 		(net 1)
 	)
+	(segment
+		(start 69.0875 82.55)
+		(end 49.5 82.55)
+		(width 0.2)
+		(layer "F.Cu")
+		(net 6)
+	)
+	(segment
+		(start 49.5 82.55)
+		(end 49.5 21.2)
+		(width 0.2)
+		(layer "F.Cu")
+		(net 6)
+	)
+	(segment
+		(start 49.5 21.2)
+		(end 27.05 21.2)
+		(width 0.2)
+		(layer "F.Cu")
+		(net 6)
+	)
+	(segment
+		(start 27.05 21.2)
+		(end 27.05 20)
+		(width 0.2)
+		(layer "F.Cu")
+		(net 6)
+	)
+	(segment
+		(start 114.04 5.11)
+		(end 139.5 5.11)
+		(width 0.2)
+		(layer "F.Cu")
+		(net 6)
+	)
+	(segment
+		(start 139.5 5.11)
+		(end 139.5 94.8)
+		(width 0.2)
+		(layer "F.Cu")
+		(net 6)
+	)
+	(segment
+		(start 122.65 94.8)
+		(end 140.475 94.8)
+		(width 0.2)
+		(layer "F.Cu")
+		(net 6)
+	)
+	(segment
+		(start 140.475 96.095)
+		(end 140.475 94.8)
+		(width 0.2)
+		(layer "F.Cu")
+		(net 6)
+	)
+	(segment
+		(start 122.65 94.8)
+		(end 122.65 96.095)
+		(width 0.2)
+		(layer "F.Cu")
+		(net 6)
+	)
+	(segment
+		(start 122.65 96.095)
+		(end 123.525 96.095)
+		(width 0.2)
+		(layer "F.Cu")
+		(net 6)
+	)
+	(segment
+		(start 125.225 90)
+		(end 125.225 94.8)
+		(width 0.2)
+		(layer "F.Cu")
+		(net 6)
+	)
+	(segment
+		(start 131.225 90)
+		(end 131.225 94.8)
+		(width 0.2)
+		(layer "F.Cu")
+		(net 6)
+	)
+	(segment
+		(start 135.525 99.905)
+		(end 135.525 101.975)
+		(width 0.2)
+		(layer "F.Cu")
+		(net 18)
+	)
+	(segment
+		(start 135.525 101.975)
+		(end 131.975 101.975)
+		(width 0.2)
+		(layer "F.Cu")
+		(net 18)
+	)
+	(segment
+		(start 140.475 99.905)
+		(end 140.475 101.975)
+		(width 0.2)
+		(layer "F.Cu")
+		(net 18)
+	)
+	(segment
+		(start 140.475 101.975)
+		(end 141.975 101.975)
+		(width 0.2)
+		(layer "F.Cu")
+		(net 18)
+	)
+	(segment
+		(start 128.475 99.905)
+		(end 128.475 101.975)
+		(width 0.2)
+		(layer "F.Cu")
+		(net 18)
+	)
+	(segment
+		(start 128.475 101.975)
+		(end 131.975 101.975)
+		(width 0.2)
+		(layer "F.Cu")
+		(net 18)
+	)
+	(segment
+		(start 128.475 97.365)
+		(end 130.475 97.365)
+		(width 0.2)
+		(layer "F.Cu")
+		(net 18)
+	)
+	(segment
+		(start 130.475 97.365)
+		(end 130.475 101.975)
+		(width 0.2)
+		(layer "F.Cu")
+		(net 18)
+	)
+	(segment
+		(start 126.775 90)
+		(end 126.775 89)
+		(width 0.2)
+		(layer "F.Cu")
+		(net 18)
+	)
+	(segment
+		(start 126.775 89)
+		(end 121.975 89)
+		(width 0.2)
+		(layer "F.Cu")
+		(net 18)
+	)
+	(segment
+		(start 121.975 89)
+		(end 121.975 91.975)
+		(width 0.2)
+		(layer "F.Cu")
+		(net 18)
+	)
+	(segment
+		(start 132.775 90)
+		(end 132.775 91.975)
+		(width 0.2)
+		(layer "F.Cu")
+		(net 18)
+	)
+	(segment
+		(start 132.775 91.975)
+		(end 131.975 91.975)
+		(width 0.2)
+		(layer "F.Cu")
+		(net 18)
+	)
+	(segment
+		(start 140.9625 107)
+		(end 140.9625 111.975)
+		(width 0.2)
+		(layer "F.Cu")
+		(net 18)
+	)
+	(segment
+		(start 140.9625 111.975)
+		(end 141.975 111.975)
+		(width 0.2)
+		(layer "F.Cu")
+		(net 18)
+	)
+	(segment
+		(start 124.8625 107.95)
+		(end 135.0375 107.95)
+		(width 0.2)
+		(layer "F.Cu")
+		(net 24)
+	)
+	(segment
+		(start 135.0375 107.95)
+		(end 135.0375 107)
+		(width 0.2)
+		(layer "F.Cu")
+		(net 24)
+	)
 	(via
