File: hardware/pcb/chip_module.kicad_sch (KiCad schematic)
At the start: 201 parts, among them J12 BTB_DAUGHTER

Commit message: test+fix: generator capstone gate (catches 3 real drifts), security-guard tests, head sheet re-baselined (round-9 audit)
THE CAPSTONE -- tests/test_generator_freshness.py now runs the REAL
generator in a temp copy of the committed inputs and compares pure-text
surfaces against BOTH committed boards: schematic instances (symbol/
position/value/footprint), label positions, no_connect markers, board
placement and every pad's net -- no kicad-cli/pcbnew needed, so CI runs
it (it skips only when the system footprint library is absent). Its
first runs caught three real drifts:

1. C87's footprint header used the full 'Capacitor_SMD:C_1206_3216Metric'
   while the generator and all 134 siblings emit the bare name -- aligned
   to the repo convention.
2. The model's ancient '"": "GND"' keys (U3 + UE0-2) netted numberless
   sub-pads that are F.Paste/F.Mask apertures with NO copper: KiCad
   discards those nets at load, the committed boards ship them netless,
   and the comments claimed 'EP copper floats' (false -- the real EP
   copper is pad 33, already netted). Keys removed, comments corrected;
   the emitter now matches what KiCad itself normalises to.
3. THE HEAD SHEET WAS STALE: the head PCB, the generator model and the
   docs all carry the ADR-0009 removable-die socket
   (qssc:ChipSocket_2.54_DET) while chip_module.kicad_sch still described
   the directly-soldered die -- footprint property pointing at the DIE
   footprint, so 'Update PCB from Schematic' would have swapped the
   socket out. The byte-for-byte freeze to the repair baseline is what
   hid it. The sheet is regenerated and the gate re-baselined as
   test_head_sheet_matches_the_socket_design (digest pin + refdes set
   vs baseline + Uchip's documented lib_id/value/footprint swap).

Also in this round:
- Security-guard branches now TESTED (they were never entered: the suite
  runs local by design): _is_local's peer-only rules (incl. forged XFF
  refusal), fpga_command's localhost guard (403 remote / 503-o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
Parts:
- removed Uchip: QSSC_Chip_DET, qssc:QSSC_Chip_DET, symbol qssc:QSSC_Chip_DET
- added Uchip: ChipSocket_2.54_DET, qssc:ChipSocket_2.54_DET, symbol qssc:ChipSocket_2.54_DET
Connections:
- net DET_IN0: now also Uchip.DET0
- net DET_IN1: now also Uchip.DET1
- net DET_IN10: now also Uchip.DET10
- net DET_IN11: now also Uchip.DET11
- net DET_IN12: now also Uchip.DET12
- net DET_IN13: now also Uchip.DET13
- net DET_IN14: now also Uchip.DET14
- net DET_IN15: now also Uchip.DET15
- net DET_IN16: now also Uchip.DET16
- net DET_IN17: now also Uchip.DET17
- net DET_IN18: now also Uchip.DET18
- net DET_IN19: now also Uchip.DET19
- net DET_IN2: now also Uchip.DET2
- net DET_IN20: now also Uchip.DET20
- net DET_IN21: now also Uchip.DET21
- net DET_IN22: now also Uchip.DET22
- net DET_IN23: now also Uchip.DET23
- net DET_IN24: now also Uchip.DET24
- net DET_IN25: now also Uchip.DET25
- net DET_IN26: now also Uchip.DET26
- net DET_IN27: now also Uchip.DET27
- net DET_IN28: now also Uchip.DET28
- net DET_IN29: now also Uchip.DET29
- net DET_IN3: now also Uchip.DET3
- net DET_IN30: now also Uchip.DET30
- net DET_IN31: now also Uchip.DET31
- net DET_IN32: now also Uchip.DET32
- net DET_IN33: now also Uchip.DET33
- net DET_IN34: now also Uchip.DET34
- net DET_IN35: now also Uchip.DET35
- net DET_IN36: now also Uchip.DET36
- net DET_IN37: now also Uchip.DET37
- net DET_IN38: now also Uchip.DET38
- net DET_IN39: now also Uchip.DET39
- net DET_IN4: now also Uchip.DET4
- net DET_IN40: now also Uchip.DET40
- net DET_IN41: now also Uchip.DET41
- net DET_IN42: now also Uchip.DET42
- net DET_IN43: now also Uchip.DET43
- net DET_IN44: now also Uchip.DET44
- net DET_IN45: now also Uchip.DET45
- net DET_IN46: now also Uchip.DET46
- net DET_IN47: now also Uchip.DET47
- net DET_IN48: now also Uchip.DET48
- net DET_IN49: now also Uchip.DET49
- net DET_IN5: now also Uchip.DET5
- net DET_IN50: now also Uchip.DET50
- net DET_IN51: now also Uchip.DET51
- net DET_IN52: now also Uchip.DET52
- net DET_IN53: now also Uchip.DET53
- net DET_IN54: now also Uchip.DET54
- net DET_IN55: now also Uchip.DET55
- net DET_IN56: now also Uchip.DET56
- net DET_IN57: now also Uchip.DET57
- net DET_IN58: now also Uchip.DET58
- net DET_IN59: now also Uchip.DET59
- net DET_IN6: now also Uchip.DET6
- net DET_IN60: now also Uchip.DET60
- net DET_IN61: now also Uchip.DET61
- net DET_IN62: now also Uchip.DET62
- net DET_IN63: now also Uchip.DET63
- net DET_IN7: now also Uchip.DET7
- net DET_IN8: now also Uchip.DET8
- net DET_IN9: now also Uchip.DET9
- net DET_REF: now also Uchip.DET_COMMON
Changed lines of the file:
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@@
 	)
 	(symbol
-		(lib_id "qssc:QSSC_Chip_DET")
+		(lib_id "qssc:ChipSocket_2.54_DET")
 		(at 80 55 0)
 		(unit 1)
@@
 			)
 		)
-		(property "Value" "QSSC_Chip_DET"
+		(property "Value" "ChipSocket_2.54_DET"
 			(at 80 57 0)
 			(effects
@@
 			)
 		)
-		(property "Footprint" "qssc:QSSC_Chip_DET"
+		(property "Footprint" "qssc:ChipSocket_2.54_DET"
 			(at 80 55 0)
 			(effects
